File: TRC2026_1/TRC2026.kicad_pcb (KiCad board)
At the start: 2 copper layers, 79 x 180 mm, 42 parts, among them J1 Conn_01x04_Pin, J10 Conn_01x07_Pin, J11 Conn_01x04_Pin, J12 Conn_01x07_Pin, J13 Conn_01x04_Pin, J14 Conn_01x04_Pin, J15 Conn_01x04_Pin, J16 Conn_01x04_Pin, J17 Conn_01x04_Pin, J18 Conn_01x04_Pin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

Commit message: 回路図変えたよ
Routing:
- net GND: track 231.0 -> 279.6 mm, vias 19 -> 27
- net LED4: track 87.3 -> 82.2 mm, vias 1 -> 3
- net RX1: track 129.1 -> 131.4 mm, vias 1 -> 3

Commit message: 基板をめちゃめちゃ修正しました
Parts:
- added G***: LOGO, LOGO, F.Cu at (143.0, 125.5)
- added J6: Conn_01x04_Pin, Connector_PinHeader_2.54mm:PinHeader_1x04_P2.54mm_Vertical, F.Cu at (134.5, 42.6)
- D10, D11, D12, D13, D14, D9: footprint KiCad_UCLAMP3381:UCLAMP3381PTFT -> KiCad_TVS:SOD2513X114N
- J1, J15, J16, J17: value Conn_01x04_Pin -> 2F接続
- J10: value Conn_01x07_Pin -> メモリ
- J11: value Conn_01x04_Pin -> BNO055
- J12: value Conn_01x07_Pin -> 気温気圧高度センサ
- J22: value Conn_01x12_Pin -> LoRa
- J7: value Conn_01x04_Pin -> GPS
- moved D13 0.57 mm to (137.5, 27.0), turned to -90 degrees
- moved D11 0.51 mm to (145.5, 40.0), turned to 180 degrees
- moved J4 0.50 mm to (79.0, 106.3)
- moved R1 0.50 mm to (138.5, 87.1)
- moved D12 0.07 mm to (145.5, 42.5), turned to 180 degrees
- turned D10 to 180 degrees
- turned D14 to -90 degrees
- turned D9 to 180 degrees
Routing:
- net GND: track 279.6 -> 355.4 mm, vias 27 -> 38
- net +24V: track 122.1 -> 196.1 mm, vias 2 -> 12
- net +5V: track 398.4 -> 413.7 mm, vias 1 -> 2
- net BOUT1: track 37.3 -> 38.8 mm
- net SCK: track 85.9 -> 87.0 mm
- net CS: track 96.8 -> 95.8 mm
- net BIN1: track 144.5 -> 145.2 mm
- net AOUT2: track 18.5 -> 19.0 mm
- net BIN2: track 119.9 -> 119.4 mm
- net RST1: vias 5 -> 7
Other:
- board text added: "100μF"
- board text added: "TRC_Noname 1F"
