File: TRC2026_1/TRC2026.kicad_sch (KiCad schematic)
At the start: 42 parts, among them J1 Conn_01x04_Pin, J10 Conn_01x07_Pin, J11 Conn_01x04_Pin, J12 Conn_01x07_Pin, J13 Conn_01x04_Pin, J14 Conn_01x04_Pin, J15 Conn_01x04_Pin, J16 Conn_01x04_Pin, J17 Conn_01x04_Pin, J18 Conn_01x04_Pin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

Commit message: 基板をめちゃめちゃ修正しました
Parts:
- added J6: Conn_01x04_Pin, Connector_PinHeader_2.54mm:PinHeader_1x04_P2.54mm_Vertical, symbol Connector:Conn_01x04_Pin
- D10, D11, D12, D13, D14, D9: footprint KiCad_UCLAMP3381:UCLAMP3381PTFT -> KiCad_TVS:SOD2513X114N
- J1, J15, J16, J17: value Conn_01x04_Pin -> 2F接続
- J10: value Conn_01x07_Pin -> メモリ
- J11: value Conn_01x04_Pin -> BNO055
- J12: value Conn_01x07_Pin -> 気温気圧高度センサ
- J22: value Conn_01x12_Pin -> LoRa
- J7: value Conn_01x04_Pin -> GPS
Connections:
- net +24V: now also J6.1 (Pin_1)
- net GND: now also J6.4 (Pin_4)
- no-connect marks 58 -> 60
Changed lines of the file:
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@@
 	)
 	(no_connect
+		(at 246.38 114.3)
+	)
+	(no_connect
 		(at 229.87 139.7)
 	)
@@
 	)
 	(no_connect
+		(at 246.38 116.84)
+	)
+	(no_connect
 		(at 25.4 55.88)
 	)
@@
 			)
 		)
-		(property "Value" "Conn_01x07_Pin"
+		(property "Value" "メモリ"
 			(at 139.7 45.72 90)
 			(effects
@@
 			)
 		)
-		(property "Footprint" "KiCad_UCLAMP3381:UCLAMP3381PTFT"
+		(property "Footprint" "KiCad_TVS:SOD2513X114N"
 			(at -4.75 177.8 0)
 			(effects
@@
 			)
 		)
-		(property "Value" "Conn_01x04_Pin"
+		(property "Value" "GPS"
 			(at 132.334 33.274 0)
 			(effects
@@
 			)
 		)
-		(property "Value" "Conn_01x04_Pin"
+		(property "Value" "2F接続"
 			(at 289.814 103.124 0)
 			(effects
@@
 			)
 		)
-		(property "Footprint" "KiCad_UCLAMP3381:UCLAMP3381PTFT"
+		(property "Footprint" "KiCad_TVS:SOD2513X114N"
 			(at 4.14 180.34 0)
 			(effects
@@
 	)
 	(symbol
+		(lib_id "power:+24V")
+		(at 246.38 111.76 0)
+		(unit 1)
+		(exclude_from_sim no)
+		(in_bom yes)
+		(on_board yes)
+		(dnp no)
+		(fields_autoplaced yes)
+		(property "Reference" "#PWR047"
+			(at 246.38 115.57 0)
+			(effects
+				(font
+					(size 1.27 1.27)
+				)
+				(hide yes)
+			)
+		)
+		(property "Value" "+24V"
+			(at 246.38 106.68 0)
+			(effects
+				(font
+					(size 1.27 1.27)
+				)
+			)
+		)
+		(property "Footprint" ""
+			(at 246.38 111.76 0)
+			(effects
+				(font
+					(size 1.27 1.27)
+				)
+				(hide yes)
+			)
+		)
+		(property "Datasheet" ""
+			(at 246.38 111.76 0)
+			(effects
+				(font
+					(size 1.27 1.27)
+				)
+				(hide yes)
+			)
+		)
+		(property "Description" "Power symbol creates a global label with name \"+24V\""
+			(at 246.38 111.76 0)
+			(effects
+				(font
+					(size 1.27 1.27)
+				)
+				(hide yes)
+			)
+		)
+		(pin "1"
+		)
+		(instances
+			(project ""
+				(path "/de8f0bed-146c-45b2-86fe-01234c757410"
+					(reference "#PWR047")
+					(unit 1)
+				)
+			)
+		)
+	)
+	(symbol
 		(lib_id "power:+5V")
 		(at 91.44 30.48 0)
@@
 			)
 		)
-		(property "Footprint" "KiCad_UCLAMP3381:UCLAMP3381PTFT"
+		(property "Footprint" "KiCad_TVS:SOD2513X114N"
 			(at 37.16 185.42 0)
 			(effects
@@
 	)
 	(symbol
+		(lib_id "power:GND")
+		(at 246.38 119.38 0)
+		(unit 1)
+		(exclude_from_sim no)
+		(in_bom yes)
+		(on_board yes)
+		(dnp no)
+		(fields_autoplaced yes)
+		(property "Reference" "#PWR038"
+			(at 246.38 125.73 0)
+			(effects
+				(font
+					(size 1.27 1.27)
+				)
+				(hide yes)
+			)
+		)
+		(property "Value" "GND"
+			(at 246.38 124.46 0)
+			(effects
+				(font
+					(size 1.27 1.27)
+				)
+			)
+		)
+		(property "Footprint" ""
+			(at 246.38 119.38 0)
+			(effects
+				(font
+					(size 1.27 1.27)
+				)
+				(hide yes)
+			)
+		)
+		(property "Datasheet" ""
+			(at 246.38 119.38 0)
+			(effects
+				(font
+					(size 1.27 1.27)
+				)
+				(hide yes)
+			)
+		)
+		(property "Description" "Power symbol creates a global label with name \"GND\" , ground"
+			(at 246.38 119.38 0)
+			(effects
+				(font
+					(size 1.27 1.27)
+				)
+				(hide yes)
+			)
+		)
+		(pin "1"
+		)
+		(instances
+			(project "TRC2026"
+				(path "/de8f0bed-146c-45b2-86fe-01234c757410"
+					(reference "#PWR038")
+					(unit 1)
+				)
+			)
+		)
+	)
+	(symbol
 		(lib_id "UCLAMP3381P_TFT:UCLAMP3381P.TFT")
 		(at 50.8 167.64 270)
@@
 			)
 		)
-		(property "Footprint" "KiCad_UCLAMP3381:UCLAMP3381PTFT"
+		(property "Footprint" "KiCad_TVS:SOD2513X114N"
 			(at -42.85 180.34 0)
 			(effects
@@
 			)
 		)
-		(property "Value" "Conn_01x04_Pin"
+		(property "Value" "2F接続"
 			(at 272.034 103.124 0)
 			(effects
@@
 			)
 		)
-		(property "Footprint" "KiCad_UCLAMP3381:UCLAMP3381PTFT"
+		(property "Footprint" "KiCad_TVS:SOD2513X114N"
 			(at 51.13 182.88 0)
 			(effects
@@
 			)
 		)
-		(property "Value" "Conn_01x12_Pin"
+		(property "Value" "LoRa"
 			(at 31.75 53.3399 0)
 			(effects
@@
 	)
 	(symbol
+		(lib_id "Connector:Conn_01x04_Pin")
+		(at 241.3 114.3 0)
+		(unit 1)
+		(exclude_from_sim no)
+		(in_bom yes)
+		(on_board yes)
+		(dnp no)
+		(property "Reference" "J6"
+			(at 241.554 100.584 0)
+			(effects
+				(font
+					(size 1.27 1.27)
+				)
+			)
+		)
+		(property "Value" "Conn_01x04_Pin"
+			(at 241.554 103.124 0)
+			(effects
+				(font
+					(size 1.27 1.27)
+				)
+			)
+		)
+		(property "Footprint" "Connector_PinHeader_2.54mm:PinHeader_1x04_P2.54mm_Vertical"
+			(at 241.3 114.3 0)
+			(effects
+				(font
+					(size 1.27 1.27)
+				)
+				(hide yes)
+			)
+		)
+		(property "Datasheet" "~"
+			(at 241.3 114.3 0)
+			(effects
+				(font
+					(size 1.27 1.27)
+				)
+				(hide yes)
+			)
+		)
+		(property "Description" "Generic connector, single row, 01x04, script generated"
+			(at 241.3 114.3 0)
+			(effects
+				(font
+					(size 1.27 1.27)
+				)
+				(hide yes)
+			)
+		)
+		(pin "2"
+		)
+		(pin "3"
+		)
+		(pin "1"
+		)
+		(pin "4"
+		)
+		(instances
+			(project "TRC2026"
+				(path "/de8f0bed-146c-45b2-86fe-01234c757410"
+					(reference "J6")
+					(unit 1)
+				)
+			)
+		)
+	)
+	(symbol
 		(lib_id "power:+5V")
 		(at 140.97 118.11 0)
@@
 			)
 		)
-		(property "Value" "Conn_01x04_Pin"
+		(property "Value" "2F接続"
 			(at 308.864 103.124 0)
 			(effects
@@
 			)
 		)
-		(property "Value" "Conn_01x04_Pin"
+		(property "Value" "BNO055"
 			(at 145.415 16.51 0)
 			(effects
@@
 			)
 		)
-		(property "Footprint" "KiCad_UCLAMP3381:UCLAMP3381PTFT"
+		(property "Footprint" "KiCad_TVS:SOD2513X114N"
 			(at -51.74 177.8 0)
 			(effects
@@
 			)
 		)
-		(property "Value" "Conn_01x07_Pin"
+		(property "Value" "気温気圧高度センサ"
 			(at 99.06 40.64 90)
 			(effects
@@
 			)
 		)
-		(property "Value" "Conn_01x04_Pin"
+		(property "Value" "2F接続"
 			(at 255.524 103.124 0)
 			(effects
