File: TRC2026_2/TRC2026_2.kicad_sch (KiCad schematic)
At the start: 31 parts, among them J1 Conn_01x02_Pin, J15 Conn_01x04_Pin, J16 デジタル電圧計(測定), J17 デジタル電圧計(電力供給), J2 Conn_01x04_Pin, J3 Conn_01x04_Pin, J4 Conn_01x04_Pin, J5 Conn_01x04_Pin, SW1 SW_SPST, SW2 SW_SPDT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

Commit message: 基板をめちゃめちゃ修正しました
Parts:
- added J6: Conn_01x04_Pin, Connector_PinHeader_2.54mm:PinHeader_1x04_P2.54mm_Vertical, symbol Connector:Conn_01x04_Pin
Connections:
- net +24V: now also J6.1 (Pin_1)
- net +5V: now also J6.2 (Pin_2), J6.3 (Pin_3)
- net GND: now also J6.4 (Pin_4)
