File: TRC2027/TRC2027main/TRC2027main.kicad_sch (KiCad schematic)
At the start: 50 parts, among them J1 Power_conn(XT90), J10 Memory, J11 BNO055, J12 Temperature, pressure, and al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, J13 Conn_01x03_Pin, J14 Conn_01x04_Pin, J15 Conn_01x04_Pin, J16 Conn_01x04_Pin, J17 Conn_01x04_Pin, J18 Conn_01x04_Pin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

Commit message: add LTE_Module
Parts:
- added D10, D11, D12, D13, D5, D6, D7, D9: UCLAMP3381P.TFT, UCLAMP3381PTFT, symbol UCLAMP3381P_TFT:UCLAMP3381P.TFT
- added J20: Conn_01x10_Pin, symbol Connector:Conn_01x10_Pin
Connections:
- net GND: now also J19.6 (Pin_6), D10.2, D11.2, D12.2, D13.2, D5.2, D6.2, D7.2, D9.2, J20.10 (Pin_10), J20.8 (Pin_8), J20.9 (Pin_9)
- net RX: now also D7.1
- net RX2: now also J19.8 (Pin_8)
- net SCL: now also D10.1, D13.1, D5.1
- net SDA: now also D11.1, D12.1, D6.1
- net TX: now also D9.1
- net TX2: now also J19.7 (Pin_7)
- net RESET: now reaches A1.31 (GPIO26_ADC0)
- net RESET: now also J19.4 (Pin_4)
- net PWRKEY: now reaches A1.32 (GPIO27_ADC1)
- net PWRKEY: now also J19.5 (Pin_5)
- no-connect marks 31 -> 43
Other:
- moved on the sheet: C3, J14, J15, J16, J8, J9
