File: TRC2027/TRC2027main/TRC2027main.kicad_pcb (KiCad board)
At the start: 2 copper layers, 120 x 278.8 mm, 76 parts, among them IC1 MCP23017-E_SP, J1 Power_conn(XT90), J10 Memory, J11 BNO055, J12 Temperature, pressure, and al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, J13 Conn_01x03_Pin, J14 Conn_01x04_Pin, J15 Conn_01x04_Pin, J16 Conn_01x04_Pin, J17 Conn_01x04_Pin, J18 Conn_01x04_Pin, J19 Conn_01x12_Pin, J2 電圧計_測定, J20 Conn_01x10_Pin, J21 Conn_01x04_Pin, J22 XH_Moter_Output, J23 XH_Moter_Output, J24 Conn_01x04_Pin, J25 Conn_01x04_Pin, J26 Conn_01x03_Pin, J27 Conn_01x03_Pin, J28 Conn_01x03_Pin, J3 電圧計_電源, J4 XH_Moter_Output, J5 XH_Moter_Output, J6 Conn_01x07_Pin, J7 GPS, J8 Conn_01x08_Pin, J9 Conn_01x08_Pin, SW1 SW_SPST, U1 DCDC, U2 DRV8262DDWR, U3 DRV8262DDWR, U4 DRV8262DDWR, U5 DRV8262DDWR

Commit message: add
Parts:
- removed A1: RaspberryPi_Pico, Module:RaspberryPi_Pico_Common_Unspecified
- removed C10: 100u, Capacitor_THT:CP_Radial_D8.0mm_P3.50mm
- removed C3: 47u, Capacitor_THT:CP_Radial_D5.0mm_P2.00mm
- removed D10, D11, D12, D13, D3, D4, D5, D6, D7, D9: UCLAMP3381P.TFT, KiCad_UCLAMP3381:UCLAMP3381PTFT
- removed IC1: MCP23017-E_SP, KiCad_MCP23017:DIP794W56P254L3486H508Q28N
- removed J10: Memory, Connector_PinSocket_2.54mm:PinSocket_1x07_P2.54mm_Vertical
- removed J11: BNO055, Connector_PinSocket_2.54mm:PinSocket_1x04_P2.54mm_Vertical
- removed J12: Temperature, pressure, and altitude sensor, Connector_PinSocket_2.54mm:PinSocket_1x07_P2.54mm_Vertical
- removed J13: Conn_01x03_Pin, Connector_PinHeader_2.54mm:PinHeader_1x03_P2.54mm_Vertical
- removed J14, J15, J17, J18, J21, J24, J25: Conn_01x04_Pin, Connector_JST:JST_XH_B4B-XH-A_1x04_P2.50mm_Vertical
- removed J16: Conn_01x04_Pin, Connector_PinHeader_2.54mm:PinHeader_1x04_P2.54mm_Vertical
- removed J19: Conn_01x12_Pin, Connector_PinHeader_2.54mm:PinHeader_1x12_P2.54mm_Vertical
- removed J20: Conn_01x10_Pin, Connector_PinHeader_2.54mm:PinHeader_1x10_P2.54mm_Vertical
- removed J6: Conn_01x07_Pin, Connector_PinHeader_2.54mm:PinHeader_1x07_P2.54mm_Vertical
- removed J7: GPS, Connector_PinSocket_2.54mm:PinSocket_1x04_P2.54mm_Vertical
- removed J8, J9: Conn_01x08_Pin, Connector_PinHeader_2.54mm:PinHeader_1x08_P2.54mm_Vertical
- removed R10: 75, Resistor_THT:R_Axial_DIN0207_L6.3mm_D2.5mm_P10.16mm_Horizontal
- removed R11: 10k, Resistor_THT:R_Axial_DIN0207_L6.3mm_D2.5mm_P10.16mm_Horizontal
- removed R4, R9: 330, Resistor_THT:R_Axial_DIN0207_L6.3mm_D2.5mm_P10.16mm_Horizontal
- removed R5, R6, R7, R8: 10, Resistor_THT:R_Axial_DIN0207_L6.3mm_D2.5mm_P10.16mm_Horizontal
- removed S1: ST12-303FCG, KiCad_ST12:ST12303FCG
- added G***: LOGO, LOGO, F.Cu at (172.2, 160.8)
- added J30: Conn_01x20_Pin, Connector_JST:JST_XH_B20B-XH-A_1x20_P2.50mm_Vertical, F.Cu at (265.0, 41.8)
- moved J3 131.1 mm to (166.0, 39.2), turned to 90 degrees
- moved PS1 120.3 mm to (188.8, 37.8), turned to 180 degrees
- moved J2 119.8 mm to (166.0, 47.8), turned to 90 degrees
- moved J28 39.3 mm to (260.2, 34.5), turned to 0 degrees
- moved C11 25.6 mm to (252.3, 91.5)
- moved C1 16.8 mm to (175.5, 48.5)
- moved J4 11.8 mm to (262.0, 122.0), turned to 0 degrees
- moved J22 10.8 mm to (261.8, 95.5), turned to 0 degrees
- moved J23 9.33 mm to (261.8, 102.5), turned to 0 degrees
- moved J5 7.85 mm to (261.8, 109.5), turned to 0 degrees
- moved J26 4.81 mm to (265.0, 149.8)
- moved D1 4.80 mm to (175.5, 129.3)
- moved C2 4.76 mm to (199.0, 88.0)
- moved J27 4.60 mm to (265.0, 129.2)
- moved C4 3.75 mm to (185.0, 47.7)
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Routing:
- net +5V: track 0.00 -> 574.2 mm, vias 0 -> 4
- net GND: track 0.00 -> 326.2 mm, vias 0 -> 28
- net +3.3V: track 0.00 -> 262.1 mm, vias 0 -> 8
- net +24V: track 0.00 -> 241.9 mm, vias 0 -> 1
- net PWM: track 0.00 -> 102.3 mm, vias 0 -> 3
- net BnFAULT: track 0.00 -> 97.5 mm, vias 0 -> 3
- net CIN1: track 0.00 -> 90.4 mm, vias 0 -> 6
- net AIN2: track 0.00 -> 85.0 mm, vias 0 -> 8
- net PWM2: track 0.00 -> 82.4 mm, vias 0 -> 3
- net BIN2: track 0.00 -> 78.8 mm, vias 0 -> 5
- net BIN1: track 0.00 -> 77.3 mm, vias 0 -> 4
- net CnFAULT: track 0.00 -> 75.9 mm, vias 0 -> 3
- net COUT1: track 0.00 -> 74.3 mm, vias 0 -> 1
- net COUT2: track 0.00 -> 71.2 mm
- net AnFAULT: track 0.00 -> 67.0 mm, vias 0 -> 2
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- added copper zone on B.Cu, net GND
- added copper zone on F.Cu, net GND
Other:
- board size 120 x 278.8 mm -> 126.6 x 279 mm
- board text added: "TRC2027_MainBoard 1F_Ver.1"

Commit message: Add positions.csv file with component placements and orientations
Parts:
- removed C5: 0.1μF, Capacitor_SMD:C_0603_1608Metric
- removed J2: 電圧計_測定, Connector_JST:JST_XH_B2B-XH-A_1x02_P2.50mm_Vertical
- removed J3: 電圧計_電源, Connector_JST:JST_XH_B2B-XH-A_1x02_P2.50mm_Vertical
- removed R13: 0.33Ω_金属皮膜, Resistor_THT:R_Axial_DIN0516_L15.5mm_D5.0mm_P20.32mm_Horizontal
- added C5_0.1u: 0.1μF, Capacitor_SMD:C_0603_1608Metric, F.Cu at (190.3, 71.5)
- added 測定電圧: 電圧計_測定, Connector_JST:JST_XH_B2B-XH-A_1x02_P2.50mm_Vertical, F.Cu at (169.5, 159.8)
- added 電源供給: 電圧計_電源, Connector_JST:JST_XH_B2B-XH-A_1x02_P2.50mm_Vertical, F.Cu at (178.1, 159.8)
- C7: value 100u -> C7_100u
- DMoter: renamed from J22; value XH_Moter_Output -> DMoter
- J28: value Conn_01x03_Pin -> Servo_1
- U1: value DCDC -> ~; footprint LMR38025:LMR -> LM70880Module:LM70880Module
- moved PS1 111.9 mm to (173.2, 148.6), turned to 0 degrees
- moved C4 104.5 mm to (167.4, 150.7), turned to 180 degrees
- moved G*** 88.2 mm to (260.4, 158.3), turned to 90 degrees
- moved C1 51.6 mm to (169.3, 99.7), turned to 180 degrees
- moved D2 38.8 mm to (187.5, 161.6)
- moved U1 27.1 mm to (177.2, 38.2), turned to 0 degrees
- moved D1 22.4 mm to (165.1, 109.4)
- moved R3 13.1 mm to (163.2, 122.7)
- moved J1 7.20 mm to (187.5, 140.7)
- moved C6 3.25 mm to (169.3, 106.8), turned to -90 degrees
- moved F2 2.60 mm to (188.0, 110.2)
- moved R1 2.45 mm to (179.6, 121.5)
- moved D8 2.38 mm to (183.9, 98.0)
- moved SW1 2.35 mm to (186.9, 88.8)
- moved R2 0.90 mm to (166.3, 122.7)
- renumbered J4 to AMoter, J23 to CMoter, J27 to Servo_2, J26 to Servo_3
Connections:
- C4 pad 1: Net-(U1-EN) -> +24V
- U1 pad 2: GND -> +24V
- U1 pad 3: unconnected-(U1-PG-Pad3) -> GND
- U1 pad 4: unconnected-(U1-NC-Pad4) -> +5V
Routing:
- net +24V: track 241.9 -> 321.3 mm, vias 1 -> 3
- net Net-(U1-EN): track 28.8 -> 0.00 mm
- net +3.3V: track 262.1 -> 287.7 mm, vias 8 -> 6
- net +BATT: track 36.4 -> 60.8 mm
- net GND: track 326.2 -> 316.8 mm
- net GND1: track 19.1 -> 11.3 mm
- net Net-(D8-K): track 22.1 -> 28.3 mm
- net +5VD: track 10.9 -> 14.5 mm
- net +5V: track 574.2 -> 573.5 mm
- net Net-(R1-Pad2): track 4.27 -> 3.58 mm
- net Net-(MD1-TRIM): track 5.16 -> 4.53 mm
Other:
- board size 126.6 x 279 mm -> 107 x 137.5 mm
- board text added: "BMoter"
- board text added: "TRC2027 MainBoard_1F_Ver.1"
- board text removed: "TRC2027_MainBoard 1F_Ver.1"
