File: TRC2027/TRC2027main/TRC2027main_ver2.kicad_pcb (KiCad board)
At the start: 4 copper layers, 107 x 157.5 mm, 37 parts, among them J1 Power_conn(XT90), J2 電圧計_測定, J22 D_Moter, J23 XH_Moter_Output, J26_Servo Conn_01x03_Pin, J27_Servo Conn_01x03_Pin, J28 servo, J3 電圧計_電源, J30 Conn_01x20_Pin, J4 A_Moter, J5 B_Moter, SW1 SW_SPST, U2 DRV8262DDWR, U3 DRV8262DDWR, U4 DRV8262DDWR, U5 DRV8262DDWR

Commit message: add
Parts:
- added C1: 470u, Capacitor_THT:CP_Radial_D12.5mm_P5.00mm, F.Cu at (113.8, 150.3)
- J22: value D_Moter -> DMoter
- J28: value servo -> Conn_01x03_Pin
- J4: value A_Moter -> AMoter
- J5: value B_Moter -> BMoter
- moved J1 18.6 mm to (101.8, 153.7), turned to 90 degrees
- renumbered J23 to CMoter, J26_Servo to J26, J27_Servo to J27
Routing:
- net +5V: track 175.9 -> 249.6 mm
- net +BATT: track 16.4 -> 19.6 mm
