File: TRC2027/DRV8262DDWModule/DRV8262DDWModule.kicad_pcb (KiCad board)
At the start: 2 copper layers, 45 x 31.5 mm, 10 parts, among them J1 XT30, J2 XT30, J3 Conn_01x05_Pin, U1 DRV8262DDWR_Module

Commit message: add
Parts:
- added D1: LED, LED_THT:LED_D5.0mm, F.Cu at (155.4, 107.6)
- added R2: 4.7k, Resistor_THT:R_Axial_DIN0207_L6.3mm_D2.5mm_P10.16mm_Horizontal, F.Cu at (140.2, 110.8)
- U1: value DRV8262DDWR_Module -> DRV8262DDWR
Routing:
- net /VM: track 80.6 -> 90.7 mm
- net Net-(D1-A): track 0.00 -> 5.28 mm
