File: TRC2027/TRC2027main2/TRC2027main2.kicad_pcb (KiCad board)
At the start: 2 copper layers, 29 parts, among them J10 Memory, J11 BNO055, J12 Temperature, pressure, and al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, J13 Conn_01x03_Pin, J14 Conn_01x04_Pin, J15 Conn_01x04_Pin, J16 Conn_01x04_Pin, J17 Conn_01x04_Pin, J18 Conn_01x04_Pin, J19 Conn_01x12_Pin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

Commit message: Add positions.csv file with component placements and orientations
Parts:
- added ?: , , F.Cu at (175.1, 131.6)
- added ?: , , F.Cu at (157.1, 131.6)
- added D10: UCLAMP3381P.TFT, KiCad_UCLAMP3381:UCLAMP3381PTFT, F.Cu at (122.0, 57.1)
- added D11: UCLAMP3381P.TFT, KiCad_UCLAMP3381:UCLAMP3381PTFT, F.Cu at (122.0, 53.9)
- added D12: UCLAMP3381P.TFT, KiCad_UCLAMP3381:UCLAMP3381PTFT, F.Cu at (220.1, 110.7)
- added D13: UCLAMP3381P.TFT, KiCad_UCLAMP3381:UCLAMP3381PTFT, F.Cu at (220.2, 107.8)
- added D3: UCLAMP3381P.TFT, KiCad_UCLAMP3381:UCLAMP3381PTFT, F.Cu at (166.3, 92.1)
- added D4: UCLAMP3381P.TFT, KiCad_UCLAMP3381:UCLAMP3381PTFT, F.Cu at (163.4, 92.1)
- added D5: UCLAMP3381P.TFT, KiCad_UCLAMP3381:UCLAMP3381PTFT, F.Cu at (136.4, 67.0)
- added D6: UCLAMP3381P.TFT, KiCad_UCLAMP3381:UCLAMP3381PTFT, F.Cu at (132.4, 67.0)
- added D7: UCLAMP3381P.TFT, KiCad_UCLAMP3381:UCLAMP3381PTFT, F.Cu at (169.6, 52.8)
- added D9: UCLAMP3381P.TFT, KiCad_UCLAMP3381:UCLAMP3381PTFT, F.Cu at (169.6, 50.0)
- added G***: LOGO, LOGO, F.Cu at (141.6, 143.2)
- added IC1: MCP23017-E_SP, KiCad_MCP23017:DIP794W56P254L3486H508Q28N, F.Cu at (184.1, 119.7)
- added S1: ST12-303FCG, KiCad_ST12:ST12303FCG, F.Cu at (133.5, 87.2)
- J16: footprint Connector_PinHeader_2.54mm:PinHeader_1x04_P2.54mm_Vertical -> Connector_JST:JST_XH_B4B-XH-A_1x04_P2.50mm_Vertical
- J7: value GPS -> BNO055
- moved J7 187.7 mm to (248.9, 129.4), turned to 90 degrees
- moved J11 186.7 mm to (256.5, 121.6), turned to -90 degrees
- moved J20 182.3 mm to (266.5, 81.1)
- moved J13 161.6 mm to (230.5, 124.7)
- moved J9 151.1 mm to (224.2, 97.8)
- moved A1 145.0 mm to (186.4, 73.6)
- moved J19 141.2 mm to (230.1, 76.1)
- moved J17 138.5 mm to (168.2, 139.6), turned to 180 degrees
- moved J8 137.0 mm to (200.7, 115.5), turned to 180 degrees
- moved J6 130.1 mm to (199.1, 124.3)
- moved J12 129.4 mm to (178.1, 145.5), turned to 90 degrees
- moved J10 123.8 mm to (192.8, 111.3)
- moved J30 115.0 mm to (119.5, 109.2), turned to 90 degrees
- moved J18 106.3 mm to (158.6, 96.8)
- moved J25 104.1 mm to (158.0, 61.0)
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Connections:
- C3 pad 1: +5V -> +3.3V
- J16 pad 2: +5V -> +3.3V
Routing:
- net +5V: track 0.00 -> 387.7 mm, vias 0 -> 3
- net GND: track 0.00 -> 386.6 mm, vias 0 -> 30
- net SCL: track 0.00 -> 313.0 mm, vias 0 -> 7
- net SDA: track 0.00 -> 310.9 mm, vias 0 -> 10
- net +3.3V: track 0.00 -> 275.6 mm, vias 0 -> 3
- net TX2: track 0.00 -> 135.6 mm, vias 0 -> 4
- net RX2: track 0.00 -> 129.8 mm, vias 0 -> 4
- net RX1: track 0.00 -> 102.0 mm, vias 0 -> 1
- net TX1: track 0.00 -> 96.9 mm
- net DIN2: track 0.00 -> 95.4 mm, vias 0 -> 2
- net DIN1: track 0.00 -> 86.7 mm, vias 0 -> 1
- net LEDSW: track 0.00 -> 86.0 mm
- net PWM3: track 0.00 -> 84.0 mm, vias 0 -> 1
- net PWM2: track 0.00 -> 81.1 mm, vias 0 -> 3
- net PWRKEY: track 0.00 -> 78.3 mm, vias 0 -> 4
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- added copper zone on B.Cu, net GND
- added copper zone on F.Cu, net GND
Other:
- board outline added: 153 x 100 mm
- board text added: "Camera"
- board text added: "Camera2"
- board text added: "FullColorLED"
- board text added: "GPS"
- board text added: "LTE"
- board text added: "LiDAR"
- board text added: "LoRa"
- board text added: "NFC/Felica"
- board text added: "TRC2027 MainBoard_2F_Ver.1"
- board text added: "気温気圧"
