File: TRC2027/TRC2027main2/TRC2027main2.kicad_pcb (KiCad board)
At the start: 2 copper layers, 153 x 100 mm, 44 parts, among them IC1 MCP23017-E_SP, J10 Memory, J11 BNO055, J12 Temperature, pressure, and al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, J13 Conn_01x03_Pin, J14 Conn_01x04_Pin, J15 Conn_01x04_Pin, J16 Conn_01x04_Pin, J17 Conn_01x04_Pin, J18 Conn_01x04_Pin, J19 Conn_01x12_Pin, J20 Conn_01x10_Pin, J21 Conn_01x04_Pin, J24 Conn_01x04_Pin, J25 Conn_01x04_Pin, J30 Conn_01x20_Pin, J6 Conn_01x07_Pin, J7 BNO055, J8 Conn_01x08_Pin, J9 Conn_01x08_Pin

Commit message: add kind GPS file
Parts:
- moved J11 10.9 mm to (248.9, 129.4), turned to 90 degrees
- moved J7 7.93 mm to (248.9, 121.5)
Connections:
- J8 pad 6: unconnected-(J8-Pin_6-Pad6) -> RST1
- J8 pad 7: RST1 -> unconnected-(J8-Pin_7-Pad7)
Routing:
- net +3.3V: track 275.6 -> 265.9 mm
- net GND: track 386.6 -> 394.5 mm
- net SCL: track 313.0 -> 308.2 mm, vias 7 -> 8
- net SDA: track 310.9 -> 306.7 mm, vias 10 -> 9

Commit message: add
Parts:
- added R1: 4.7k, Resistor_THT:R_Axial_DIN0207_L6.3mm_D2.5mm_P10.16mm_Horizontal, F.Cu at (173.3, 71.5)
- added R2: 4.7k, Resistor_THT:R_Axial_DIN0207_L6.3mm_D2.5mm_P10.16mm_Horizontal, F.Cu at (170.1, 70.5)
- moved ? 26.6 mm to (148.5, 132.9)
- moved ? 26.6 mm to (130.5, 132.9)
- moved J17 2.62 mm to (168.2, 142.2)
Connections:
- A1 pad 20: unconnected-(A1-GPIO15-Pad20)_1 -> M0
- A1 pad 29: unconnected-(A1-GPIO22-Pad29) -> M1
- J6 pad 1: unconnected-(J6-Pin_1-Pad1) -> M0
- J6 pad 2: unconnected-(J6-Pin_2-Pad2) -> M1
Routing:
- net M1: track 0.00 -> 65.9 mm, vias 0 -> 3
- net +3.3V: track 265.9 -> 311.9 mm, vias 3 -> 5
- net M0: track 0.00 -> 45.4 mm, vias 0 -> 1
- net GND: track 394.5 -> 380.1 mm
- net SDA: track 306.7 -> 316.9 mm
- net SCL: track 308.2 -> 314.7 mm
- net +5V: track 387.7 -> 392.3 mm
Other:
- board text added: "3.3V ×"
- board text added: "TRC2027 MainBoard_2F_Ver.2"
- board text removed: "TRC2027 MainBoard_2F_Ver.1"
