File: TRC2027/TRC2027main2/TRC2027main2.kicad_sch (KiCad schematic)
At the start: 41 parts, among them IC1 MCP23017-E_SP, J10 Memory, J11 BNO055, J12 Temperature, pressure, and al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, J13 Conn_01x03_Pin, J14 Conn_01x04_Pin, J15 Conn_01x04_Pin, J16 Conn_01x04_Pin, J17 Conn_01x04_Pin, J18 Conn_01x04_Pin, J19 Conn_01x12_Pin, J20 Conn_01x10_Pin, J21 Conn_01x04_Pin, J24 Conn_01x04_Pin, J25 Conn_01x04_Pin, J30 Conn_01x20_Pin, J6 Conn_01x07_Pin, J7 BNO055, J8 Conn_01x08_Pin, J9 Conn_01x08_Pin

Commit message: add kind GPS file
Connections:
- net RST1: now also J8.6 (Pin_6); no longer J8.7 (Pin_7)
Changed lines of the file:
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@@
+	)
+	(no_connect
+		(at 20.32 58.42)
 	)
 	(no_connect
@@
 	)
 	(no_connect
-		(at 20.32 60.96)
-	)
-	(no_connect
 		(at 66.04 149.86)
 	)
@@
 		)
 	)
+	(global_label "RST1"
+		(shape input)
+		(at 20.32 60.96 180)
+		(fields_autoplaced yes)
+		(effects
+			(font
+				(size 1.27 1.27)
+			)
+			(justify right)
+		)
+		(property "Intersheetrefs" "${INTERSHEET_REFS}"
+			(at 12.6782 60.96 0)
+			(effects
+				(font
+					(size 1.27 1.27)
+				)
+				(justify right)
+				(hide yes)
+			)
+		)
+	)
 	(global_label "RX"
 		(shape input)
@@
 				(hide yes)
 			)
-		)
-	)
-	(global_label "RST1"
-		(shape input)
-		(at 20.32 58.42 180)
-		(fields_autoplaced yes)
-		(effects
-			(font
-				(size 1.27 1.27)
-			)
-			(justify right)
-		)
-		(property "Intersheetrefs" "${INTERSHEET_REFS}"
-			(at 12.6782 58.42 0)
-			(effects
-				(font
-					(size 1.27 1.27)
-				)
-				(justify right)
-				(hide yes)
-			)

Commit message: add
Parts:
- added R1, R2: 4.7k, Resistor_THT:R_Axial_DIN0207_L6.3mm_D2.5mm_P10.16mm_Horizontal, symbol Device:R
Connections:
- net +3.3V: now also R1.1, R2.1
- net SCL: now also R1.2
- net SDA: now also R2.2
- net M0: now reaches J6.1 (Pin_1)
- net M0: now also A1.20 (GPIO15)
- net M1: now reaches J6.2 (Pin_2)
- net M1: now also A1.29 (GPIO22)
- no-connect marks 46 -> 42
