File: TRC2027/LM70880Module/LM70880.kicad_pcb (KiCad board)
At the start: 2 copper layers, 30.2 x 29 mm, 27 parts, among them J1 Conn_01x02_Pin, J2 Conn_01x02_Pin, U1 LM70880RRXR

Commit message: add Artwork
Parts:
- removed R8: 1, Resistor_SMD:R_0603_1608Metric
- removed R9: 5m, Resistor_SMD:R_1206_3216Metric
- added R4: 9.53k, Resistor_SMD:R_0805_2012Metric, F.Cu at (103.9, 75.2)
- C1: value 4.7u -> 15u; footprint Capacitor_SMD:C_0805_2012Metric -> Capacitor_THT:CP_Radial_D10.0mm_P5.00mm
- C10: value 47n -> 10u; footprint Capacitor_SMD:C_0603_1608Metric -> Capacitor_SMD:C_0805_2012Metric
- C11, C12, C13, C14: value 47u -> 10u; footprint Capacitor_SMD:C_0603_1608Metric -> Capacitor_SMD:C_0805_2012Metric
- C2, C6: value 4.7u -> 0.1u; footprint Capacitor_SMD:C_0805_2012Metric -> Capacitor_SMD:C_0603_1608Metric
- C4: value 4.7u -> 3.3n; footprint Capacitor_SMD:C_0805_2012Metric -> Capacitor_SMD:C_0603_1608Metric
- C5: value 0.1u -> 22p
- C7: value 6.8n -> 1u
- C8: value 47p -> 47n
- C9: value 0.1u -> 10u; footprint Capacitor_SMD:C_0603_1608Metric -> Capacitor_SMD:C_0805_2012Metric
- L1: value 3.3u -> 8.2u; footprint KiCadLIB_SMMS1050-5R6M:SMMS10505R6M -> Inductor_SMD:L_Wuerth_WE-PD-Typ-LS_Handsoldering
- R1: value 100k -> 237k; footprint Resistor_SMD:R_0603_1608Metric -> Resistor_SMD:R_0805_2012Metric
- R2: value 20.5k -> 19.6k; footprint Resistor_SMD:R_0603_1608Metric -> Resistor_SMD:R_0805_2012Metric
- R5: value 5.76k -> 29.4k
- R6: value 29.4k -> 54.9k
- R7: value 54.9k -> 5m; footprint Resistor_SMD:R_0603_1608Metric -> Resistor_SMD:R_1206_3216Metric
- moved C12 22.1 mm to (99.9, 78.9), turned to 90 degrees
- moved C14 21.6 mm to (97.9, 78.9), turned to 90 degrees
- moved C13 20.0 mm to (101.9, 78.9), turned to 90 degrees
- moved C11 18.3 mm to (103.9, 78.9), turned to 90 degrees
- moved G*** 15.3 mm to (113.6, 62.6)
- moved C7 13.7 mm to (109.3, 74.2), turned to 90 degrees
- moved R2 12.4 mm to (95.0, 64.2), turned to 90 degrees
- moved C10 12.0 mm to (105.9, 78.9), turned to 90 degrees
- moved R7 10.9 mm to (111.8, 79.8), turned to 180 degrees
- moved C4 9.67 mm to (106.3, 74.2), turned to -90 degrees
- moved C5 8.18 mm to (107.8, 74.2), turned to -90 degrees
- moved R1 7.35 mm to (95.0, 67.7), turned to 90 degrees
- moved C1 7.29 mm to (102.8, 67.5), turned to 0 degrees
- moved R5 7.21 mm to (95.3, 78.8), turned to 180 degrees
- moved R3 5.08 mm to (101.5, 74.7), turned to -90 degrees
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Connections:
- C10 pad 1: Net-(U1-CBOOT) -> +5V
- C10 pad 2: Net-(C10-Pad2) -> GND
- C3 pad 1: +24V -> GND
- C3 pad 2: GND -> Net-(U1-VCC)
- C4 pad 1: +24V -> GND
- C4 pad 2: GND -> Net-(C4-Pad2)
- C5 pad 1: +24V -> GND
- C5 pad 2: GND -> Net-(U1-EXTCOMP)
- C6 pad 1: Net-(U1-VCC) -> Net-(U1-PFM_SYNCIN)
- C7 pad 1: GND -> +5V
- C7 pad 2: Net-(C7-Pad2) -> GND
- C8 pad 1: GND -> Net-(U1-CBOOT)
- C8 pad 2: Net-(U1-EXTCOMP) -> Net-(U1-SW1)
- C9 pad 1: GND -> +5V
- C9 pad 2: Net-(U1-VDDA) -> GND
- R3 pad 1: Net-(U1-VDDA) -> Net-(U1-PFM_SYNCIN)
- R5 pad 1: Net-(C7-Pad2) -> Net-(U1-CONFIG)
- R5 pad 2: Net-(U1-EXTCOMP) -> GND
- R6 pad 1: GND -> Net-(U1-RT)
- R6 pad 2: Net-(U1-CONFIG) -> GND
- R7 pad 1: GND -> Net-(U1-ISNS+)
- R7 pad 2: Net-(U1-RT) -> +5V
- U1 pad 18: Net-(U1-VDDA) -> Net-(U1-PFM_SYNCIN)
- U1 pad 8: GND -> Net-(U1-PFM_SYNCIN)
Routing:
- net GND: track 14.7 -> 54.8 mm, vias 30 -> 23
- net +24V: track 69.9 -> 33.2 mm
- net Net-(U1-SW1): track 28.1 -> 48.4 mm, vias 4 -> 3
- net Net-(C10-Pad2): track 12.1 -> 0.00 mm, vias 2 -> 0
- net +5V: track 58.6 -> 70.3 mm
- net Net-(U1-PFM_SYNCIN): track 0.00 -> 9.80 mm, vias 0 -> 2
- net Net-(U1-EN_UVLO): track 3.86 -> 11.8 mm, vias 0 -> 2
- net Net-(U1-VCC): track 2.03 -> 9.31 mm, vias 0 -> 2
- net Net-(C7-Pad2): track 5.30 -> 0.00 mm, vias 2 -> 0
- net Net-(U1-VDDA): track 4.79 -> 0.00 mm
- net Net-(U1-CBOOT): track 1.52 -> 5.54 mm, vias 0 -> 2
- net Net-(U1-RT): track 2.77 -> 6.66 mm
- net Net-(U1-EXTCOMP): track 8.43 -> 10.8 mm, vias 2 -> 0
- net Net-(C4-Pad2): track 0.00 -> 1.62 mm
- net Net-(U1-ISNS+): track 27.1 -> 25.6 mm, vias 0 -> 4
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Other:
- board size 30.2 x 29 mm -> 30 x 29 mm
- board text added: "LM70880"
- board text removed: "LM70880Module"
