File: TRC2027/LM70880Module/LM70880.kicad_sch (KiCad schematic)
At the start: 27 parts, among them J1 Conn_01x02_Pin, J2 Conn_01x02_Pin, U1 LM70880RRXR

Commit message: add Artwork
Parts:
- removed R8: 1, Resistor_SMD:R_0603_1608Metric, symbol Device:R
- removed R9: 5m, Resistor_SMD:R_1206_3216Metric, symbol Device:R
- C1: value 4.7u -> 15u; footprint Capacitor_SMD:C_0805_2012Metric -> Capacitor_THT:CP_Radial_D10.0mm_P5.00mm
- C10: value 47n -> 10u; footprint Capacitor_SMD:C_0603_1608Metric -> Capacitor_SMD:C_0805_2012Metric
- C11, C12, C13, C14: value 47u -> 10u; footprint Capacitor_SMD:C_0603_1608Metric -> Capacitor_SMD:C_0805_2012Metric
- C2, C6: value 4.7u -> 0.1u; footprint Capacitor_SMD:C_0805_2012Metric -> Capacitor_SMD:C_0603_1608Metric
- C4: value 4.7u -> 3.3n; footprint Capacitor_SMD:C_0805_2012Metric -> Capacitor_SMD:C_0603_1608Metric
- C5: value 0.1u -> 22p
- C7: value 6.8n -> 1u
- C8: value 47p -> 47n
- C9: value 0.1u -> 10u; footprint Capacitor_SMD:C_0603_1608Metric -> Capacitor_SMD:C_0805_2012Metric
- L1: value 3.3u -> 8.2u; footprint KiCadLIB_SMMS1050-5R6M:SMMS10505R6M -> Inductor_SMD:L_Wuerth_WE-PD-Typ-LS_Handsoldering
- R1: value 100k -> 237k; footprint Resistor_SMD:R_0603_1608Metric -> Resistor_SMD:R_0805_2012Metric
- R2: value 20.5k -> 19.6k; footprint Resistor_SMD:R_0603_1608Metric -> Resistor_SMD:R_0805_2012Metric
- R4: value 19.1k -> 9.53k; footprint Resistor_SMD:R_0603_1608Metric -> Resistor_SMD:R_0805_2012Metric
- R5: value 5.76k -> 29.4k
- R6: value 29.4k -> 54.9k
- R7: value 54.9k -> 5m; footprint Resistor_SMD:R_0603_1608Metric -> Resistor_SMD:R_1206_3216Metric
Connections:
- net +24V: no longer C3.1, C4.1, C5.1
- net +5V: now also C10.1, C7.1, C9.1, R7.2
- net GND: now also C10.2, C3.1, C4.1, C5.1, C7.2, C9.2, R5.2, R6.2; no longer C3.2, C4.2, C5.2, C7.1, C8.1, C9.1, R4.1, R6.1, R7.1, U1.8 (PFM_SYNCIN)
- net at U1.19 (VCC): now also C3.2; no longer C6.1
- net at R3.1, U1.18 (VDDA): now also C6.1, U1.8 (PFM_SYNCIN); no longer C9.2
- net at R5.1: now also U1.13 (CONFIG); no longer C7.2
- net at L1.1, U1.20 (SW1), U1.21 (SW2)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: now also C8.2
- net at L1.2, U1.11 (ISNS+): now also R7.1
- net at U1.4 (CBOOT): now also C8.1; no longer C10.1
- net at U1.14 (RT): now also R6.1; no longer R7.2
- net at R3.2, U1.16 (FB): no longer R4.2
- new net: C4.2, R4.1
- new net: C5.2, R4.2, U1.15 (EXTCOMP)
